File: 0-10V-to-4-20mA-Converter.kicad_pcb (KiCad board)
At the start: 2 copper layers, 48.7 x 24.8 mm, 15 parts, among them J1 Conn_01x02_Pin, J2 Conn_01x02_Pin, Q1 BCP56, U1 XTR116U, U2 MCP6002-I_SN

Commit message: PCB_filled
Routing:
- net /IRET_LOCAL: track 32.6 -> 36.5 mm, vias 2 -> 6
- added copper zone on B.Cu, net /IRET_LOCAL
- added copper zone on F.Cu, net /IRET_LOCAL
